File: KiCad/keyboard.sch (KiCad schematic (older format))
At the start: 130 parts

Commit message: Wired USB
Parts:
- added F?: Polyfuse, symbol Device:Polyfuse
- added USB?: Molex-0548190589, symbol random-keyboard-parts:Molex-0548190589
Connections:
- net +5V: now also F?.1
- net D+: now also USB?.3 (D+)
- net D-: now also USB?.4 (D-)
- net GND: now also USB?.1 (GND)
- new net VCC: F?.2, USB?.5 (VBUS)
Changed lines of the file:
@@
 Text GLabel 11535 10035 0    50   Input ~ 0
 D-
+$Comp
+L random-keyboard-parts:Molex-0548190589 USB?
+U 1 1 6149CA0B
+P 17820 6560
+F 0 "USB?" V 18357 6527 60  0000 C CNN
+F 1 "Molex-0548190589" V 18251 6527 60  0000 C CNN
+F 2 "" H 17820 6560 60  0001 C CNN
+F 3 "" H 17820 6560 60  0001 C CNN
+	1    17820 6560
+	0    -1   -1   0
+$EndComp
+$Comp
+L power:VCC #PWR?
+U 1 1 614EF491
+P 18550 6360
+F 0 "#PWR?" H 18550 6210 50  0001 C CNN
+F 1 "VCC" H 18567 6533 50  0000 C CNN
+F 2 "" H 18550 6360 50  0001 C CNN
+F 3 "" H 18550 6360 50  0001 C CNN
+	1    18550 6360
+	1    0    0    -1
+$EndComp
+$Comp
+L Device:Polyfuse F?
+U 1 1 614F0170
+P 19025 6360
+F 0 "F?" V 18800 6360 50  0000 C CNN
+F 1 "Polyfuse" V 18891 6360 50  0000 C CNN
+F 2 "" H 19075 6160 50  0001 L CNN
+F 3 "~" H 19025 6360 50  0001 C CNN
+	1    19025 6360
+	0    1    1    0
+$EndComp
+$Comp
+L power:+5V #PWR?
+U 1 1 614F0D68
+P 19535 6360
+F 0 "#PWR?" H 19535 6210 50  0001 C CNN
+F 1 "+5V" H 19550 6533 50  0000 C CNN
+F 2 "" H 19535 6360 50  0001 C CNN
+F 3 "" H 19535 6360 50  0001 C CNN
+	1    19535 6360
+	1    0    0    -1
+$EndComp
+Wire Wire Line
+	18120 6360 18550 6360
+Wire Wire Line
+	18550 6360 18875 6360
+Connection ~ 18550 6360
+Wire Wire Line
+	19175 6360 19535 6360
+$Comp
+L power:GND #PWR?
+U 1 1 61530793
+P 18390 6760
+F 0 "#PWR?" H 18390 6510 50  0001 C CNN
+F 1 "GND" H 18395 6587 50  0000 C CNN
+F 2 "" H 18390 6760 50  0001 C CNN
+F 3 "" H 18390 6760 50  0001 C CNN
+	1    18390 6760
+	1    0    0    -1
+$EndComp
+Wire Wire Line
+	18390 6760 18120 6760
+Text GLabel 18120 6460 2    50   Input ~ 0
+D-
+Text GLabel 18120 6560 2    50   Input ~ 0
+D+
 $EndSCHEMATC

Commit message: Assigned footprints
Parts:
- C1, C2, C3, C4, C5, C6, C7: renamed from C?; footprint (none) -> Capacitor_SMD:C_0805_2012Metric
- F1: renamed from F?; footprint (none) -> Fuse:Fuse_1206_3216Metric
- R1, R2, R3, R4: renamed from R?; footprint (none) -> Resistor_SMD:R_0805_2012Metric
- SW1: renamed from SW?; footprint (none) -> random-keyboard-parts:SKQG-1155865
- USB1: renamed from USB?; footprint (none) -> random-keyboard-parts:Molex-0548190589
- Y1: renamed from Y?; footprint (none) -> Crystal:Crystal_SMD_3225-4Pin_3.2x2.5mm
- gave numbers to parts that had none: 1
Changed lines of the file:
@@
 	13800 950  13800 1950
 $Comp
-L MCU_Microchip_ATmega:ATmega32U4-AU U?
+L MCU_Microchip_ATmega:ATmega32U4-AU U1
 U 1 1 610E833C
 P 13110 10435
-F 0 "U?" H 13110 8546 50  0000 C CNN
+F 0 "U1" H 13110 8546 50  0000 C CNN
 F 1 "ATmega32U4-AU" H 13110 8455 50  0000 C CNN
 F 2 "Package_QFP:TQFP-44_10x10mm_P0.8mm" H 13110 10435 50  0001 C CIN
@@
 $EndComp
 $Comp
-L power:+5V #PWR?
+L power:+5V #PWR0101
 U 1 1 610F8D3E
 P 13010 8510
-F 0 "#PWR?" H 13010 8360 50  0001 C CNN
+F 0 "#PWR0101" H 13010 8360 50  0001 C CNN
 F 1 "+5V" H 13025 8683 50  0000 C CNN
 F 2 "" H 13010 8510 50  0001 C CNN
@@
 	13110 8635 13010 8635
 $Comp
-L power:GND #PWR?
+L power:GND #PWR0102
 U 1 1 61108E51
 P 13010 12370
-F 0 "#PWR?" H 13010 12120 50  0001 C CNN
+F 0 "#PWR0102" H 13010 12120 50  0001 C CNN
 F 1 "GND" H 13015 12197 50  0000 C CNN
 F 2 "" H 13010 12370 50  0001 C CNN
@@
 Connection ~ 13010 12235
 $Comp
-L Device:R_Small R?
+L Device:R_Small R4
 U 1 1 6111A522
 P 14055 11035
-F 0 "R?" V 13859 11035 50  0000 C CNN
+F 0 "R4" V 13859 11035 50  0000 C CNN
 F 1 "10k" V 13950 11035 50  0000 C CNN
-F 2 "" H 14055 11035 50  0001 C CNN
+F 2 "Resistor_SMD:R_0805_2012Metric" H 14055 11035 50  0001 C CNN
 F 3 "~" H 14055 11035 50  0001 C CNN
 	1    14055 11035
@@
 $EndComp
 $Comp
-L power:GND #PWR?
+L power:GND #PWR0103
 U 1 1 6111BFFC
 P 14405 11035
-F 0 "#PWR?" H 14405 10785 50  0001 C CNN
+F 0 "#PWR0103" H 14405 10785 50  0001 C CNN
 F 1 "GND" H 14410 10862 50  0000 C CNN
 F 2 "" H 14405 11035 50  0001 C CNN
@@
 	14155 11035 14405 11035
 $Comp
-L Device:R_Small R?
+L Device:R_Small R2
 U 1 1 6114B2FB
 P 12100 9935
-F 0 "R?" V 11904 9935 50  0000 C CNN
+F 0 "R2" V 11904 9935 50  0000 C CNN
 F 1 "22" V 11995 9935 50  0000 C CNN
-F 2 "" H 12100 9935 50  0001 C CNN
+F 2 "Resistor_SMD:R_0805_2012Metric" H 12100 9935 50  0001 C CNN
 F 3 "~" H 12100 9935 50  0001 C CNN
 	1    12100 9935
@@
 $EndComp
 $Comp
-L Device:R_Small R?
+L Device:R_Small R1
 U 1 1 6114BD80
 P 11815 10035
-F 0 "R?" V 11619 10035 50  0000 C CNN
+F 0 "R1" V 11619 10035 50  0000 C CNN
 F 1 "22" V 11710 10035 50  0000 C CNN
-F 2 "" H 11815 10035 50  0001 C CNN
+F 2 "Resistor_SMD:R_0805_2012Metric" H 11815 10035 50  0001 C CNN
 F 3 "~" H 11815 10035 50  0001 C CNN
 	1    11815 10035
@@
 	11715 10035 11535 10035
 $Comp
-L Device:C_Small C?
+L Device:C_Small C7
 U 1 1 611D7131
 P 12255 10335
-F 0 "C?" H 12347 10381 50  0000 L CNN
+F 0 "C7" H 12347 10381 50  0000 L CNN
 F 1 "1uF" H 12347 10290 50  0000 L CNN
-F 2 "" H 12255 10335 50  0001 C CNN
+F 2 "Capacitor_SMD:C_0805_2012Metric" H 12255 10335 50  0001 C CNN
 F 3 "~" H 12255 10335 50  0001 C CNN
 	1    12255 10335
@@
 $EndComp
 $Comp
-L power:GND #PWR?
+L power:GND #PWR0104
 U 1 1 611D7FD2
 P 12255 10580
-F 0 "#PWR?" H 12255 10330 50  0001 C CNN
+F 0 "#PWR0104" H 12255 10330 50  0001 C CNN
 F 1 "GND" H 12260 10407 50  0000 C CNN
 F 2 "" H 12255 10580 50  0001 C CNN
@@
 	12255 10580 12255 10435
 $Comp
-L Device:C_Small C?
+L Device:C_Small C1
 U 1 1 6121BF75
 P 10155 11885
-F 0 "C?" H 10247 11931 50  0000 L CNN
+F 0 "C1" H 10247 11931 50  0000 L CNN
 F 1 "0.1uF" H 10247 11840 50  0000 L CNN
-F 2 "" H 10155 11885 50  0001 C CNN
+F 2 "Capacitor_SMD:C_0805_2012Metric" H 10155 11885 50  0001 C CNN
 F 3 "~" H 10155 11885 50  0001 C CNN
 	1    10155 11885
@@
 $EndComp
 $Comp
-L Device:C_Small C?
+L Device:C_Small C2
 U 1 1 6122C7C0
 P 10380 11885
-F 0 "C?" H 10472 11931 50  0000 L CNN
+F 0 "C2" H 10472 11931 50  0000 L CNN
 F 1 "0.1uF" H 10472 11840 50  0000 L CNN
-F 2 "" H 10380 11885 50  0001 C CNN
+F 2 "Capacitor_SMD:C_0805_2012Metric" H 10380 11885 50  0001 C CNN
 F 3 "~" H 10380 11885 50  0001 C CNN
 	1    10380 11885
@@
 $EndComp
 $Comp
-L Device:C_Small C?
+L Device:C_Small C3
 U 1 1 6122CB75
 P 10605 11885
-F 0 "C?" H 10697 11931 50  0000 L CNN
+F 0 "C3" H 10697 11931 50  0000 L CNN
 F 1 "0.1uF" H 10697 11840 50  0000 L CNN
-F 2 "" H 10605 11885 50  0001 C CNN
+F 2 "Capacitor_SMD:C_0805_2012Metric" H 10605 11885 50  0001 C CNN
 F 3 "~" H 10605 11885 50  0001 C CNN
 	1    10605 11885
@@
 $EndComp
 $Comp
-L Device:C_Small C?
+L Device:C_Small C4
 U 1 1 6122CD80
 P 10830 11885
-F 0 "C?" H 10922 11931 50  0000 L CNN
+F 0 "C4" H 10922 11931 50  0000 L CNN
 F 1 "10uF" H 10922 11840 50  0000 L CNN
-F 2 "" H 10830 11885 50  0001 C CNN
+F 2 "Capacitor_SMD:C_0805_2012Metric" H 10830 11885 50  0001 C CNN
 F 3 "~" H 10830 11885 50  0001 C CNN
 	1    10830 11885
@@
 	10490 11985 10380 11985
 $Comp
-L power:GND #PWR?
+L power:GND #PWR0105
 U 1 1 612E22E7
 P 10490 12085
-F 0 "#PWR?" H 10490 11835 50  0001 C CNN
+F 0 "#PWR0105" H 10490 11835 50  0001 C CNN
 F 1 "GND" H 10495 11912 50  0000 C CNN
 F 2 "" H 10490 12085 50  0001 C CNN
@@
 $EndComp
 $Comp
-L power:+5V #PWR?
+L power:+5V #PWR0106
 U 1 1 612E2DE1
 P 10490 11670
-F 0 "#PWR?" H 10490 11520 50  0001 C CNN
+F 0 "#PWR0106" H 10490 11520 50  0001 C CNN
 F 1 "+5V" H 10505 11843 50  0000 C CNN
 F 2 "" H 10490 11670 50  0001 C CNN
@@
 $EndComp
 $Comp
-L power:+5V #PWR?
+L power:+5V #PWR0107
 U 1 1 61309072
 P 12330 9735
-F 0 "#PWR?" H 12330 9585 50  0001 C CNN
+F 0 "#PWR0107" H 12330 9585 50  0001 C CNN
 F 1 "+5V" H 12345 9908 50  0000 C CNN
 F 2 "" H 12330 9735 50  0001 C CNN
@@
 	12510 9735 12330 9735
 $Comp
-L Device:Crystal_GND24_Small Y?
+L Device:Crystal_GND24_Small Y1
 U 1 1 6133E986
 P 11975 9235
-F 0 "Y?" V 11929 9379 50  0000 L CNN
+F 0 "Y1" V 11929 9379 50  0000 L CNN
 F 1 "Crystal_GND24_Small" V 12020 9379 50  0000 L CNN
-F 2 "" H 11975 9235 50  0001 C CNN
+F 2 "Crystal:Crystal_SMD_3225-4Pin_3.2x2.5mm" H 11975 9235 50  0001 C CNN
 F 3 "~" H 11975 9235 50  0001 C CNN
 	1    11975 9235
@@
 	12510 9335 11975 9335
 $Comp
-L Device:C_Small C?
+L Device:C_Small C5
 U 1 1 61385D79
 P 11600 9115
-F 0 "C?" V 11829 9115 50  0000 C CNN
+F 0 "C5" V 11829 9115 50  0000 C CNN
 F 1 "22pF" V 11738 9115 50  0000 C CNN
-F 2 "" H 11600 9115 50  0001 C CNN
+F 2 "Capacitor_SMD:C_0805_2012Metric" H 11600 9115 50  0001 C CNN
 F 3 "~" H 11600 9115 50  0001 C CNN
 	1    11600 9115
@@
 $EndComp
 $Comp
-L Device:C_Small C?
+L Device:C_Small C6
 U 1 1 6139971B
 P 11600 9335
-F 0 "C?" V 11829 9335 50  0000 C CNN
+F 0 "C6" V 11829 9335 50  0000 C CNN
 F 1 "22pF" V 11738 9335 50  0000 C CNN
-F 2 "" H 11600 9335 50  0001 C CNN
+F 2 "Capacitor_SMD:C_0805_2012Metric" H 11600 9335 50  0001 C CNN
 F 3 "~" H 11600 9335 50  0001 C CNN
 	1    11600 9335
@@
 $EndComp
 $Comp
-L power:GND #PWR?
+L power:GND #PWR0108
 U 1 1 613CF3CE
 P 11500 9535
-F 0 "#PWR?" H 11500 9285 50  0001 C CNN
+F 0 "#PWR0108" H 11500 9285 50  0001 C CNN
 F 1 "GND" H 11505 9362 50  0000 C CNN
 F 2 "" H 11500 9535 50  0001 C CNN
@@
 	11875 9445 11875 9535
 $Comp
-L power:GND #PWR?
+L power:GND #PWR0109
 U 1 1 6142F07A
 P 11890 8885
-F 0 "#PWR?" H 11890 8635 50  0001 C CNN
+F 0 "#PWR0109" H 11890 8635 50  0001 C CNN
 F 1 "GND" H 11895 8712 50  0000 C CNN
 F 2 "" H 11890 8885 50  0001 C CNN
@@
 $EndComp
 $Comp
-L Switch:SW_Push SW?
+L Switch:SW_Push SW1
 U 1 1 61430CED
 P 12215 8935
-F 0 "SW?" H 12215 9220 50  0000 C CNN
+F 0 "SW1" H 12215 9220 50  0000 C CNN
 F 1 "SW_Push" H 12215 9129 50  0000 C CNN
-F 2 "" H 12215 9135 50  0001 C CNN
+F 2 "random-keyboard-parts:SKQG-1155865" H 12215 9135 50  0001 C CNN
 F 3 "~" H 12215 9135 50  0001 C CNN
 	1    12215 8935
@@
 	12470 8935 12415 8935
 $Comp
-L Device:R_Small R?
+L Device:R_Small R3
 U 1 1 6146D06F
 P 12470 8500
-F 0 "R?" H 12529 8546 50  0000 L CNN
+F 0 "R3" H 12529 8546 50  0000 L CNN
 F 1 "R_Small" H 12529 8455 50  0000 L CNN
-F 2 "" H 12470 8500 50  0001 C CNN
+F 2 "Resistor_SMD:R_0805_2012Metric" H 12470 8500 50  0001 C CNN
 F 3 "~" H 12470 8500 50  0001 C CNN
 	1    12470 8500
@@
 $EndComp
 $Comp
-L power:+5V #PWR?
+L power:+5V #PWR0110
 U 1 1 6146EADF
 P 12470 8250
-F 0 "#PWR?" H 12470 8100 50  0001 C CNN
+F 0 "#PWR0110" H 12470 8100 50  0001 C CNN
 F 1 "+5V" H 12485 8423 50  0000 C CNN
 F 2 "" H 12470 8250 50  0001 C CNN
@@
 D-
 $Comp
-L random-keyboard-parts:Molex-0548190589 USB?
+L random-keyboard-parts:Molex-0548190589 USB1
 U 1 1 6149CA0B
 P 17820 6560
-F 0 "USB?" V 18357 6527 60  0000 C CNN
+F 0 "USB1" V 18357 6527 60  0000 C CNN
 F 1 "Molex-0548190589" V 18251 6527 60  0000 C CNN
-F 2 "" H 17820 6560 60  0001 C CNN
+F 2 "random-keyboard-parts:Molex-0548190589" H 17820 6560 60  0001 C CNN
 F 3 "" H 17820 6560 60  0001 C CNN
 	1    17820 6560
@@
 $EndComp
 $Comp
-L power:VCC #PWR?
+L power:VCC #PWR0111
 U 1 1 614EF491
 P 18550 6360
-F 0 "#PWR?" H 18550 6210 50  0001 C CNN
+F 0 "#PWR0111" H 18550 6210 50  0001 C CNN
 F 1 "VCC" H 18567 6533 50  0000 C CNN
 F 2 "" H 18550 6360 50  0001 C CNN
@@
 $EndComp
 $Comp
-L Device:Polyfuse F?
+L Device:Polyfuse F1
 U 1 1 614F0170
 P 19025 6360
-F 0 "F?" V 18800 6360 50  0000 C CNN
+F 0 "F1" V 18800 6360 50  0000 C CNN
 F 1 "Polyfuse" V 18891 6360 50  0000 C CNN
-F 2 "" H 19075 6160 50  0001 L CNN
+F 2 "Fuse:Fuse_1206_3216Metric" H 19075 6160 50  0001 L CNN
 F 3 "~" H 19025 6360 50  0001 C CNN
 	1    19025 6360
@@
 $EndComp
 $Comp
-L power:+5V #PWR?
+L power:+5V #PWR0112
 U 1 1 614F0D68
 P 19535 6360
-F 0 "#PWR?" H 19535 6210 50  0001 C CNN
+F 0 "#PWR0112" H 19535 6210 50  0001 C CNN
 F 1 "+5V" H 19550 6533 50  0000 C CNN
 F 2 "" H 19535 6360 50  0001 C CNN
@@
 	19175 6360 19535 6360
 $Comp
-L power:GND #PWR?
+L power:GND #PWR0113
 U 1 1 61530793
 P 18390 6760
-F 0 "#PWR?" H 18390 6510 50  0001 C CNN
+F 0 "#PWR0113" H 18390 6510 50  0001 C CNN
 F 1 "GND" H 18395 6587 50  0000 C CNN
 F 2 "" H 18390 6760 50  0001 C CNN

Commit message: Finished routing switch matrix
...I think :P
Connections:
- net +5V: no longer U1.24 (AVCC), U1.44 (AVCC)
- net GND: no longer R4.1
- net col0: now also U1.36 (PF7)
- net col1: now also U1.32 (PC7)
- net col10: now also U1.21 (PD3)
- net col11: now also U1.20 (PD2)
- net col12: now also U1.19 (PD1)
- net col13: now also U1.11 (PB3)
- net col14: now also U1.18 (PD0)
- net col2: now also U1.31 (PC6)
- net col3: now also U1.30 (PB6)
- net col4: now also U1.29 (PB5)
- net col5: now also U1.28 (PB4)
- net col6: now also U1.27 (PD7)
- net col7: now also U1.26 (PD6)
- net col8: now also U1.25 (PD4)
- net col9: now also U1.22 (PD5)
- net row0: now also U1.37 (PF6)
- net row1: now also U1.38 (PF5)
- net row2: now also U1.39 (PF4)
- net row3: now also U1.40 (PF1)
- net row4: now also U1.41 (PF0)
- net at U1.33 (~HWB~/PE2): no longer R4.2
- new net: U1.24 (AVCC), U1.44 (AVCC)
Changed lines of the file:
@@
 EESchema Schematic File Version 4
+LIBS:keyboard-cache
 EELAYER 30 0
 EELAYER END
@@
 $EndComp
 Wire Wire Line
-	13210 8635 13110 8635
-Wire Wire Line
 	13010 8635 13010 8510
-Connection ~ 13010 8635
-Connection ~ 13110 8635
-Wire Wire Line
-	13110 8635 13010 8635
 $Comp
 L power:GND #PWR0102
@@
 Wire Wire Line
 	13010 12235 13010 12370
-Connection ~ 13010 12235
 $Comp
 L Device:R_Small R4
@@
 $EndComp
 Wire Wire Line
-	13710 11035 13955 11035
-Wire Wire Line
-	14155 11035 14405 11035
+	13710 11035 13910 11035
+Wire Wire Line
+	14155 11035 14210 11035
 $Comp
 L Device:R_Small R2
@@
 Text GLabel 18120 6560 2    50   Input ~ 0
 D+
+Text GLabel 13710 11335 2    50   Input ~ 0
+row4
+Text GLabel 13710 11435 2    50   Input ~ 0
+row3
+Text GLabel 13710 11535 2    50   Input ~ 0
+row2
+Text GLabel 13710 11635 2    50   Input ~ 0
+row1
+Text GLabel 13710 11735 2    50   Input ~ 0
+row0
+Text GLabel 13710 9935 2    50   Input ~ 0
+col1
+Text GLabel 13710 9835 2    50   Input ~ 0
+col2
+Text GLabel 13710 9535 2    50   Input ~ 0
+col3
+Text GLabel 13710 9435 2    50   Input ~ 0
+col4
+Text GLabel 13710 9335 2    50   Input ~ 0
+col5
+Wire Wire Line
+	14310 11035 14405 11035
+Wire Wire Line
+	13010 8635 13110 8635
+Connection ~ 13010 8635
+Connection ~ 13010 12235
+Text GLabel 13710 10835 2    50   Input ~ 0
+col6
+Text GLabel 13710 10735 2    50   Input ~ 0
+col7
+Text GLabel 13710 10535 2    50   Input ~ 0
+col8
+Text GLabel 13710 11835 2    50   Input ~ 0
+col0
+Text GLabel 13710 10635 2    50   Input ~ 0
+col9
+Text GLabel 13710 10435 2    50   Input ~ 0
+col10
+Text GLabel 13710 10335 2    50   Input ~ 0
+col11
+Text GLabel 13710 10235 2    50   Input ~ 0
+col12
+Text GLabel 13710 10135 2    50   Input ~ 0
+col14
+Text GLabel 13710 9235 2    50   Input ~ 0
+col13
 $EndSCHEMATC
