File: KiCad/keyboard.kicad_pcb (KiCad board)
At the start: 2 copper layers, 293.7 x 135.7 mm, 132 parts, among them SW1 SW_Push, U1 ATmega32U4-AU, Y1 Crystal_GND24_Small

Commit message: Component placement tweaked
Parts:
- moved C1 2.25 mm to (42.1, 7.94)
- moved R3 2.25 mm to (38.9, 7.94)
- moved R2 0.51 mm to (31.0, 3.17)
Changed lines of the file:
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@@
   )
   (module Resistor_SMD:R_0805_2012Metric (layer B.Cu)
-    (at 37.30625 6.35 270)
+    (at 38.89375 7.9375 270)
     (descr "Resistor SMD 0805 (2012 Metric), square (rectangular) end terminal, IPC_7351 nominal, (Body size source: https://docs.google.com/spreadsheets/d/1BsfQQcO9C6DZCsRaXUlFlo91Tg2WpOkGARC1WS5S8t0/edit?usp=sharing), generated with kicad-footprint-generator")
     (tags resistor)
@@
   )
   (module Resistor_SMD:R_0805_2012Metric (layer B.Cu)
-    (at 30.449 3.175 90)
+    (at 30.95625 3.175 90)
     (descr "Resistor SMD 0805 (2012 Metric), square (rectangular) end terminal, IPC_7351 nominal, (Body size source: https://docs.google.com/spreadsheets/d/1BsfQQcO9C6DZCsRaXUlFlo91Tg2WpOkGARC1WS5S8t0/edit?usp=sharing), generated with kicad-footprint-generator")
     (tags resistor)
@@
   )
   (module Capacitor_SMD:C_0805_2012Metric (layer B.Cu)
-    (at 40.48125 6.35 90)
-    (descr "Capacitor SMD 0805 (2012 Metric), square (rectangular) end terminal, IPC_7351 nominal, (Body size source: https://docs.google.com/spreadsheets/d/1BsfQQcO9C6DZCsRaXUlFlo91Tg2WpOkGARC1WS5S8t0/edit?usp=sharing), generated with kicad-footprint-generator")
-    (tags capacitor)
+    (at 42.06875 7.9375 90)
+    (descr "Capacitor SMD 0805 (2012 Metric), square (rectangular) end terminal, IPC_7351 nominal, (Body size source: https://docs.google.com/spreadsheets/d/1BsfQQcO9C6DZCsRaXUlFlo91Tg2WpOkGARC1WS5S8t0/edit?usp=sharing), generated with kicad-footprint-generator")
+    (tags capacitor)

Commit message: Routed traces (except for switch matrix)
Parts:
- SW1, USB1: moved to B.Cu
- moved R1 3.17 mm to (30.2, 3.17)
- moved R4 2.38 mm to (60.3, 19.8)
- moved R2 1.59 mm to (32.5, 3.17)
- moved C5 1.59 mm to (55.2, 1.81)
- moved C6 1.59 mm to (45.7, 1.81)
- moved Y1 1.59 mm to (50.4, 1.81)
- turned SW1 to 180 degrees
Routing:
- net +5V: track 0.00 -> 142.7 mm, vias 0 -> 5
- net GND: track 0.00 -> 74.4 mm
- net Net-(R3-Pad2): track 0.00 -> 27.1 mm, vias 0 -> 2
- net Net-(R1-Pad1): track 0.00 -> 22.9 mm
- net Net-(R2-Pad1): track 0.00 -> 21.7 mm
- net Net-(C6-Pad2): track 0.00 -> 12.6 mm
- net VCC: track 0.00 -> 12.1 mm
- net Net-(C5-Pad2): track 0.00 -> 9.92 mm
- net D+: track 0.00 -> 4.42 mm
- net D-: track 0.00 -> 4.41 mm
- net Net-(R4-Pad2): track 0.00 -> 4.08 mm
Other:
- net class Default: trace_width 0.25 -> 0.254
- net class Power added: clearance 0.2, trace_width 0.381, via_dia 0.8, via_drill 0.4

Commit message: Finished routing switch matrix
...I think :P
Connections:
- R4 pad 1: GND -> Net-(R4-Pad1)
- U1 pad 11: Net-(U1-Pad11) -> col13
- U1 pad 18: Net-(U1-Pad18) -> col14
- U1 pad 19: Net-(U1-Pad19) -> col12
- U1 pad 20: Net-(U1-Pad20) -> col11
- U1 pad 21: Net-(U1-Pad21) -> col10
- U1 pad 22: Net-(U1-Pad22) -> col9
- U1 pad 24: +5V -> Net-(U1-Pad24)
- U1 pad 25: Net-(U1-Pad25) -> col8
- U1 pad 26: Net-(U1-Pad26) -> col7
- U1 pad 27: Net-(U1-Pad27) -> col6
- U1 pad 28: Net-(U1-Pad28) -> col5
- U1 pad 29: Net-(U1-Pad29) -> col4
- U1 pad 30: Net-(U1-Pad30) -> col3
- U1 pad 31: Net-(U1-Pad31) -> col2
- U1 pad 32: Net-(U1-Pad32) -> col1
- U1 pad 33: Net-(R4-Pad2) -> Net-(U1-Pad33)
- U1 pad 36: Net-(U1-Pad36) -> col0
- U1 pad 37: Net-(U1-Pad37) -> row0
- U1 pad 38: Net-(U1-Pad38) -> row1
- U1 pad 39: Net-(U1-Pad39) -> row2
- U1 pad 40: Net-(U1-Pad40) -> row3
- U1 pad 41: Net-(U1-Pad41) -> row4
- U1 pad 44: +5V -> Net-(U1-Pad24)
Routing:
- net row3: track 0.00 -> 393.2 mm
- net row2: track 0.00 -> 375.0 mm
- net row4: track 0.00 -> 368.9 mm
- net row1: track 0.00 -> 356.1 mm
- net row0: track 0.00 -> 336.9 mm
- net col13: track 0.00 -> 316.9 mm, vias 0 -> 1
- net col12: track 0.00 -> 311.6 mm
- net col11: track 0.00 -> 291.4 mm
- net col14: track 0.00 -> 275.4 mm
- net col10: track 0.00 -> 251.2 mm
- net col9: track 0.00 -> 231.0 mm
- net col8: track 0.00 -> 205.9 mm
- net col7: track 0.00 -> 204.6 mm
- net col6: track 0.00 -> 167.1 mm
- net col5: track 0.00 -> 147.7 mm
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
Commit message: Finalized PCB
Parts:
- moved D_11 103.5 mm to (310.9, 125.1)
- moved D_37 103.5 mm to (287.1, 163.2)
- moved K_41 103.5 mm to (104.8, 181.8)
- moved K_44 103.5 mm to (173.8, 181.8)
- moved K_50 103.5 mm to (288.1, 181.8)
- moved K_9 103.5 mm to (264.3, 124.6)
- moved C2 103.5 mm to (116.3, 97.5)
- moved C3 103.5 mm to (110.5, 111.1)
- moved C4 103.5 mm to (96.8, 106.4)
- moved C5 103.5 mm to (110.7, 89.1)
- moved C7 103.5 mm to (97.1, 101.7)
- moved D_0 103.5 mm to (101.4, 125.1)
- moved D_1 103.5 mm to (120.4, 125.1)
- moved D_10 103.5 mm to (291.9, 125.1)
- moved D_12 103.5 mm to (330.0, 125.1)
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Connections:
- R4 pad 1: Net-(R4-Pad1) -> GND
- U1 pad 24: Net-(U1-Pad24) -> +5V
- U1 pad 33: Net-(U1-Pad33) -> Net-(R4-Pad2)
- U1 pad 44: Net-(U1-Pad24) -> +5V
Routing:
- net +5V: track 142.7 -> 106.4 mm
- net GND: track 74.4 -> 107.0 mm
- added copper zone on B.Cu, net GND
Other:
- board text added: "betaboz V1"
